Commit message: gripper

File: urdf/hek_4L_1.0.urdf (robot description, URDF)
Before this commit: robot hek, 9 links, 8 joints
Links:
- link base_footprint: geometry visual mesh filename=package://arm_model/stl/hek_4L_1.0/base.stl scale=0.001 0.001 0.001
- link finger_L: geometry visual mesh filename=package://arm_model/stl/graboid/finger_L.stl scale=0.001 0.001 0.001
- link finger_R: geometry visual mesh filename=package://arm_model/stl/graboid/finger_R.stl scale=0.001 0.001 0.001
- link forearm: geometry visual mesh filename=package://arm_model/stl/hek_4L_1.0/forearm.stl scale=0.001 0.001 0.001
- link gear_assembly: geometry visual mesh filename=package://arm_model/stl/graboid/gear_assembly.stl scale=0.001 0.001 0.001
- link tool_zero: geometry visual mesh filename=package://arm_model/stl/hek_4L_1.0/tool_zero.stl scale=0.001 0.001 0.001
- link upper_arm: geometry visual mesh filename=package://arm_model/stl/hek_4L_1.0/upper_arm.stl scale=0.001 0.001 0.001
- link wrist_link: geometry visual mesh filename=package://arm_model/stl/hek_4L_1.0/wrist.stl scale=0.001 0.001 0.001
